Commit message: adding leg to jey robot

File: robots/jey_description/urdf/jey.urdf (robot description, URDF)
Before this commit: robot jey, 7 links, 6 joints
Links:
- added link calf, mass 0.047629; collision mesh filename=package://example-robot-data/robots/jey_description/meshes/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 scale=1 1 1; visual mesh filename=package://example-robot-data/robots/jey_description/meshes/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 scale=1 1 1
- added link thigh, mass 0.047629; collision mesh filename=package://example-robot-data/robots/jey_description/meshes/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 scale=1 1 1; visual mesh filename=package://example-robot-data/robots/jey_description/meshes/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 scale=1 1 1
Joints:
- added joint calf_joint: type revolute, parent thigh, child calf, origin xyz=0 -0.12 0 rpy=3.141592653589793 0 0, axis 0 0 1, limit lower=-2.6 upper=-0.6 effort=140 velocity=15.55
- added joint thigh_joint: type revolute, parent trunk, child thigh, origin xyz=0 0 -0.1 rpy=1.5707963267948966 0 0, axis 0 0 1, limit lower=-1.0 upper=3.5 effort=93.33 velocity=23.32
- joint $foot_fixed: origin xyz=0 0 -0.1 rpy=0 0 0 -> xyz=0 0.12 0 rpy=0 0 0; parent trunk -> calf
