Commit message: add leg robots

File: robots/z1_5_description/urdf/z1.urdf (robot description, URDF)
Before this commit: robot z1_description, 10 links, 9 joints
Links:
- removed link link00
- removed link link01
- removed link link02
- removed link link03
- removed link link04
Joints:
- removed joint joint1
- removed joint joint2
- removed joint joint3
- removed joint joint4
- removed joint joint5
- joint base_static_joint: child link00 -> link05
