Commit message: clean closed loop kin robots

File: robots/b1_leg_FL/urdf/b1_3d.urdf (robot description, URDF)
Before this commit: robot b1_leg_description, 17 links, 16 joints
Links:
- removed link calf_loop_joint
- removed link loop_1_bar
- removed link loop_1_link
- removed link loop_2_bar
- removed link loop_2_link
- removed link loop_act_bar
- removed link loop_bar_link
- removed link reduction_loop_joint
- added link closedloop3D_1A
- added link closedloop3D_1B
- added link crank_bar2, mass 0.1; visual box size=0.01 0.01 0.043
- added link link_2_loop3D_bar3, mass 0.75; visual box size=0.01 0.01 0.3
Joints:
- removed joint calf_loop_joint
- removed joint loop_1_bar
- removed joint loop_1_calf
- removed joint loop_2_act
- removed joint loop_2_bar
- removed joint loop_act_bar
- removed joint loop_bar_act
- removed joint reduction_loop_joint
- added joint closedloop3D_1A_frame: type fixed, parent link_2_loop3D_bar3, child closedloop3D_1A, origin xyz=0 0 0.3 rpy=0 3.1415 0, axis 0 0 0
- added joint closedloop3D_1B_frame: type fixed, parent FL_calf, child closedloop3D_1B, origin xyz=0.00322198 0 0.04287912 rpy=0 0 0, axis 0 0 0
- added joint crank_bar2_thigh: type revolute, parent FL_thigh, child crank_bar2, origin xyz=0 0 -0.0515 rpy=0 0 0, axis 0 1 0, limit lower=-3.14 upper=3.14 effort=10 velocity=5
- added joint link_2_crank_bar2: type revolute, parent crank_bar2, child link_2_loop3D_bar3, origin xyz=0 0 0.043 rpy=0 0 0, axis 0 1 0, limit lower=-3.14 upper=3.14 effort=10 velocity=5
